File: mcu.kicad_sch (KiCad schematic)
At the start: 0 parts

Commit message: schema functionally done
Parts:
- added C24, C27: 1uF, Capacitor_SMD:C_0402_1005Metric, symbol Device:C
- added C25, C26, C28, C29, C30, C31, C32, C33, C34, C41: 100nF, Capacitor_SMD:C_0402_1005Metric, symbol Device:C
- added C35: 100nF, Capacitor_SMD:C_0805_2012Metric, symbol Device:C
- added C38, C39: 15pF, Capacitor_SMD:C_0805_2012Metric, symbol Device:C
- added D5: IN-S63AT5A, LED_SMD:LED_0603_1608Metric, symbol Device:LED
- added D6: RB521S30, Diode_SMD:D_SOD-523, symbol user:RB521S30
- added GP14, GP15, GP23, GP24, GP25, GP26, GP27, GP28, GP29: TestPoint_Small, TestPoint:TestPoint_Pad_D2.0mm, symbol Connector:TestPoint_Small
- added IC1: RP2040, Package_DFN_QFN:QFN-56-1EP_7x7mm_P0.4mm_EP3.2x3.2mm, symbol MCU_RaspberryPi:RP2040
- added R33, R34: 10k, Resistor_SMD:R_0805_2012Metric, symbol Device:R
- added R36, R39: 1k, Resistor_SMD:R_0805_2012Metric, symbol Device:R
- added R40, R41: 27.4, Resistor_SMD:R_0402_1005Metric, symbol Device:R
- added R42: 560R, Resistor_SMD:R_0805_2012Metric, symbol Device:R
- added R43, R44: 100R, Resistor_SMD:R_0402_1005Metric, symbol Device:R
- added R5: DNF, Resistor_SMD:R_0805_2012Metric, symbol Device:R
- added U1: W25Q64JVSSIQ, Package_SO:SOIC-8_5.23x5.23mm_P1.27mm, symbol Memory_Flash:W25Q32JVSS
- added Y2: ABM3B-12.000MHZ-10-1-U-T, Crystal:Crystal_SMD_Abracon_ABM3B-4Pin_5.0x3.2mm, symbol Device:Crystal_GND24
Connections:
- new net: GP24.1, IC1.36 (GPIO24)
- new net: GP27.1, IC1.39 (GPIO27_ADC1)
- new net: C24.1, C25.1, C26.1, IC1.23 (DVDD), IC1.45 (VREG_VOUT), IC1.50 (DVDD)
- new net: GP28.1, IC1.40 (GPIO28_ADC2)
- new net: IC1.25 (SWD), R44.2
- new net: IC1.47 (USB_DP), R40.2
- new net: GP23.1, IC1.35 (GPIO23)
- new net: GP14.1, IC1.17 (GPIO14)
- new net: GP15.1, IC1.18 (GPIO15)
- new net: IC1.24 (SWCLK), R43.2
- new net: GP25.1, IC1.37 (GPIO25)
- new net: GP26.1, IC1.38 (GPIO26_ADC0)
- new net: GP29.1, IC1.41 (GPIO29_ADC3)
- new net: IC1.46 (USB_DM), R41.2
- new net: C39.2, R39.1, Y2.3
- new net: D5.2 (A), R42.2
- new net +3V0: C27.1, C28.1, C29.1, C30.1, C31.1, C32.1, C33.1, C34.1, C35.1, D6.2 (A), IC1.1 (IOVDD), IC1.10 (IOVDD), IC1.22 (IOVDD), IC1.33 (IOVDD), IC1.42 (IOVDD), IC1.43 (ADC_AVDD), IC1.44 (VREG_IN), IC1.49 (IOVDD), R33.1, R34.1, R5.1, U1.8 (VCC)
- new net +3V3: C41.1, D6.1 (K), IC1.48 (USB_VDD)
- new net GND: C24.2, C25.2, C26.2, C27.2, C28.2, C29.2, C30.2, C31.2, C32.2, C33.2, C34.2, C35.2, C38.1, C39.1, C41.2, D5.1 (K), IC1.19 (TESTEN), IC1.57 (GND), U1.4 (GND), Y2.2, Y2.4
- new net KEY_A: IC1.9 (GPIO7)
- new net KEY_B: IC1.11 (GPIO8)
- new net KEY_C: IC1.12 (GPIO9)
- new net KEY_D: IC1.13 (GPIO10)
- new net KEY_E: IC1.14 (GPIO11)
- new net KEY_F: IC1.15 (GPIO12)
- new net LCD_COMIN: IC1.8 (GPIO6)
- new net LCD_SCLK: IC1.4 (GPIO2)
- new net LCD_SCS: IC1.7 (GPIO5)
- new net LCD_SI: IC1.5 (GPIO3)
- new net LED: IC1.6 (GPIO4), R42.1
- new net MENU: IC1.16 (GPIO13)
- new net MOUSE_1A: IC1.27 (GPIO16)
- new net MOUSE_1B: IC1.28 (GPIO17)
- new net MOUSE_2A: IC1.29 (GPIO18)
- new net MOUSE_2B: IC1.30 (GPIO19)
- new net MOUSE_3A: IC1.31 (GPIO20)
- new net MOUSE_3B: IC1.32 (GPIO21)
- new net QSPI_SCLK: IC1.52 (QSPI_SCLK), U1.6 (CLK)
- new net QSPI_SD0: IC1.53 (QSPI_SD0), U1.5 (DI(IO0))
- new net QSPI_SD1: IC1.55 (QSPI_SD1), U1.2 (DO(IO1))
- new net QSPI_SD2: IC1.54 (QSPI_SD2), U1.3 (IO2)
- new net QSPI_SD3: IC1.51 (QSPI_SD3), U1.7 (IO3)
- new net QSPI_SS: IC1.56 (QSPI_SS), R36.2, R5.2, U1.1 (~{CS})
- new net SCL: IC1.3 (GPIO1), R34.2
- new net SDA: IC1.2 (GPIO0), R33.2
- new net SWCLK: R43.1
- new net SWD: R44.1
- new net TP_RDY: IC1.34 (GPIO22)
- new net USB_D+: R40.1
- new net USB_D-: R41.1
- new net XIN: C38.2, IC1.20 (XIN), Y2.1
- new net XOUT: IC1.21 (XOUT), R39.2
- new net ~{RST}: IC1.26 (RUN)
- new net ~{USB_BOOT}: R36.1
Other:
- note added: "12MHz crystal"
- note added: "64Mbit flash memory"
- note added: "Place resistors close to MCU"
- note added: "USB termination"
- note added: "indicator LED"
- note added: "power supply"

Commit message: reannotation
Parts:
- renumbered C25 to C10, C24 to C11, C41 to C12, C27 to C13, C28 to C14, C29 to C15, C30 to C16, C31 to C17, C32 to C18, C33 to C19, C34 to C20, C38 to C6, C39 to C7, C35 to C8, C26 to C9, D5 to D7, GP14 to GP1, GP15 to GP2, GP23 to GP3, GP24 to GP4, GP25 to GP5, GP26 to GP6, GP27 to GP7, GP28 to GP8, GP29 to GP9, IC1 to IC3, R40 to R10, R41 to R11, R43 to R12, R44 to R13, R33 to R14, R34 to R15, R42 to R16, R36 to R7, R5 to R8, R39 to R9, Y2 to Y1
Other:
- moved on the sheet: C11, C13

Commit message: schematic cleanup
Parts:
- removed C10, C14, C15, C16, C17, C18, C19, C20, C9: 100nF, Capacitor_SMD:C_0402_1005Metric, symbol Device:C
- added C10, C14, C15, C16, C17, C18, C19, C20, C9: 100nF, Capacitor_SMD:C_0402_1005Metric, symbol Device:C_Small
Connections:
- net +3V0: now also C14.1, C15.1, C16.1, C17.1, C18.1, C19.1, C20.1
- net GND: now also C10.2, C14.2, C15.2, C16.2, C17.2, C18.2, C19.2, C20.2, C9.2
- net at C11.1, IC3.23 (DVDD), IC3.45 (VREG_VOUT)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: now also C10.1, C9.1
Other:
- note added: "2 x 100nF"
- note added: "7 x 100nF"
- moved on the sheet: C11, C12, C13, C6, C7, C8, D6, D7, GP1, GP2, GP3, GP4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
