File: mcu.kicad_sch (KiCad schematic)
At the start: 51 parts, among them IC3 RP2040, U1 W25Q64JVZPIQ, Y1 ABM3B-12.000MHZ-10-1-U-T

Commit message: in progress pcb
Parts:
- C6, C7, C8: footprint Capacitor_SMD:C_0805_2012Metric -> Capacitor_SMD:C_0603_1608Metric
- R14, R15, R16, R7, R8, R9: footprint Resistor_SMD:R_0805_2012Metric -> Resistor_SMD:R_0603_1608Metric
- TP28, TP29, TP30, TP43, TP44, TP45, TP46, TP47, TP48: footprint TestPoint:TestPoint_Pad_D2.0mm -> TestPoint:TestPoint_Pad_D1.0mm
- TP31: value GP02 -> GP12; footprint TestPoint:TestPoint_Pad_D2.0mm -> TestPoint:TestPoint_Pad_D1.0mm
- TP32: value GP03 -> GP13; footprint TestPoint:TestPoint_Pad_D2.0mm -> TestPoint:TestPoint_Pad_D1.0mm
- TP33: value GP04 -> GP14; footprint TestPoint:TestPoint_Pad_D2.0mm -> TestPoint:TestPoint_Pad_D1.0mm
- TP34: value GP05 -> GP15; footprint TestPoint:TestPoint_Pad_D2.0mm -> TestPoint:TestPoint_Pad_D1.0mm
- TP35: value GP08 -> GP18; footprint TestPoint:TestPoint_Pad_D2.0mm -> TestPoint:TestPoint_Pad_D1.0mm
- TP36: value GP13 -> GP19; footprint TestPoint:TestPoint_Pad_D2.0mm -> TestPoint:TestPoint_Pad_D1.0mm
- TP37: value GP14 -> GP20; footprint TestPoint:TestPoint_Pad_D2.0mm -> TestPoint:TestPoint_Pad_D1.0mm
- TP38: value GP15 -> GP21; footprint TestPoint:TestPoint_Pad_D2.0mm -> TestPoint:TestPoint_Pad_D1.0mm
- TP39: value GP16 -> GP22; footprint TestPoint:TestPoint_Pad_D2.0mm -> TestPoint:TestPoint_Pad_D1.0mm
- TP40: value GP21 -> GP23; footprint TestPoint:TestPoint_Pad_D2.0mm -> TestPoint:TestPoint_Pad_D1.0mm
- TP41: value GP26 -> GP24; footprint TestPoint:TestPoint_Pad_D2.0mm -> TestPoint:TestPoint_Pad_D1.0mm
- TP42: value GP27 -> GP25; footprint TestPoint:TestPoint_Pad_D2.0mm -> TestPoint:TestPoint_Pad_D1.0mm
Connections:
- net KEY_A: now also IC3.2 (GPIO0); no longer IC3.12 (GPIO9)
- net KEY_B: now also IC3.3 (GPIO1); no longer IC3.13 (GPIO10)
- net KEY_C: now also IC3.4 (GPIO2); no longer IC3.14 (GPIO11)
- net KEY_D: now also IC3.5 (GPIO3); no longer IC3.29 (GPIO18)
- net KEY_E: now also IC3.6 (GPIO4); no longer IC3.30 (GPIO19)
- net KEY_F: now also IC3.7 (GPIO5); no longer IC3.31 (GPIO20)
- net LCD_COMIN: now also IC3.40 (GPIO28_ADC2); no longer IC3.36 (GPIO24)
- net LCD_SCLK: now also IC3.38 (GPIO26_ADC0); no longer IC3.34 (GPIO22)
- net LCD_SCS: now also IC3.41 (GPIO29_ADC3); no longer IC3.37 (GPIO25)
- net LCD_SI: now also IC3.39 (GPIO27_ADC1); no longer IC3.35 (GPIO23)
- net MENU: now also IC3.8 (GPIO6); no longer IC3.15 (GPIO12)
- net MOUSE_1: now also IC3.11 (GPIO8); no longer IC3.8 (GPIO6)
- net MOUSE_2: now also IC3.12 (GPIO9); no longer IC3.9 (GPIO7)
- net MOUSE_3: now also IC3.13 (GPIO10); no longer IC3.40 (GPIO28_ADC2)
- net MOUSE_4: now also IC3.14 (GPIO11); no longer IC3.41 (GPIO29_ADC3)
- net SCL: now also IC3.28 (GPIO17); no longer IC3.3 (GPIO1)
- net SDA: now also IC3.27 (GPIO16); no longer IC3.2 (GPIO0)
- net TP_RDY: now also IC3.9 (GPIO7); no longer IC3.28 (GPIO17)
- net at TP35.1: now also IC3.29 (GPIO18); no longer IC3.11 (GPIO8)
- net at IC3.16 (GPIO13): now also TP32.1; no longer TP36.1
- net at TP31.1: now also IC3.15 (GPIO12); no longer IC3.4 (GPIO2)
- net at IC3.18 (GPIO15): now also TP34.1; no longer TP38.1
- net at TP42.1: now also IC3.37 (GPIO25); no longer IC3.39 (GPIO27_ADC1)
- net at TP37.1: now also IC3.31 (GPIO20); no longer IC3.17 (GPIO14)
- net at TP39.1: now also IC3.34 (GPIO22); no longer IC3.27 (GPIO16)
- net at IC3.32 (GPIO21): now also TP38.1; no longer TP40.1
- net at TP41.1: now also IC3.36 (GPIO24); no longer IC3.38 (GPIO26_ADC0)
- net at TP33.1: now also IC3.17 (GPIO14); no longer IC3.6 (GPIO4)
- new net: IC3.30 (GPIO19), TP36.1
- new net: IC3.35 (GPIO23), TP40.1
Other:
- moved on the sheet: D7, R14, R15, R16
