File: gkos_pebble.kicad_sch (KiCad schematic)
At the start: 0 parts

Commit message: power schema
Other:
- added sheet ble (ble.kicad_sch)
- added sheet inputs (inputs.kicad_sch)
- added sheet lcd (lcd.kicad_sch)
- added sheet mcu (mcu.kicad_sch)
- added sheet power (power.kicad_sch)
Changed lines of the file:
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@@
     (comment 1 "main sheet")
   )
-  (text_box "- BLE module\n- RP2040 MCU\n- NiMH charger\n- NiMH cell connection\n- 3V boost converter\n- USB-C connection + TVS\n- keyboard switches\n- mouse buttons\n- touchpad\n- memory LCD"
-    (at 24.13 153.67 0) (size 50.8 34.29)
+  (text_box "- BLE module\n- RP2040 MCU\n- USB-C connection + TVS\n- keyboard switches\n- mouse buttons\n- touchpad\n- memory LCD"
+    (at 24.13 153.67 0) (size 50.8 25.4)
     (stroke (width 0) (type default) (color 132 0 0 1))
     (fill (type color) (color 255 255 194 1))
@@
     (effects (font (size 3 3) (thickness 0.6) bold italic (color 132 0 0 1)) (justify left bottom))
   )
+  (sheet (at 127 114.3) (size 27.94 20.32) (fields_autoplaced)
+    (stroke (width 0.1524) (type solid))
+    (fill (color 255 255 194 1.0000))
+    (property "Sheetname" "mcu" (at 127 113.5884 0)
+      (effects (font (size 1.27 1.27)) (justify left bottom))
+    )
+    (property "Sheetfile" "mcu.kicad_sch" (at 127 135.2046 0)
+      (effects (font (size 1.27 1.27)) (justify left top))
+    )
+    (instances
+      (project "gkos_pebble"
+        (path "/ab6fff6e-44fa-4992-ab9d-8d9a7df4367d" (page "3"))
+      )
+    )
+  )
+  (sheet (at 92.71 72.39) (size 27.94 20.32) (fields_autoplaced)
+    (stroke (width 0.1524) (type solid))
+    (fill (color 255 255 194 1.0000))
+    (property "Sheetname" "inputs" (at 92.71 71.6784 0)
+      (effects (font (size 1.27 1.27)) (justify left bottom))
+    )
+    (property "Sheetfile" "inputs.kicad_sch" (at 92.71 93.2946 0)
+      (effects (font (size 1.27 1.27)) (justify left top))
+    )
+    (instances
+      (project "gkos_pebble"
+        (path "/ab6fff6e-44fa-4992-ab9d-8d9a7df4367d" (page "5"))
+      )
+    )
+  )
+  (sheet (at 93.98 38.1) (size 24.13 5.08) (fields_autoplaced)
+    (stroke (width 0.1524) (type solid))
+    (fill (color 255 255 194 1.0000))
+    (property "Sheetname" "power" (at 93.98 37.3884 0)
+      (effects (font (size 1.27 1.27)) (justify left bottom))
+    )
+    (property "Sheetfile" "power.kicad_sch" (at 93.98 43.7646 0)
+      (effects (font (size 1.27 1.27)) (justify left top))
+    )
+    (pin "USB_VBUS" input (at 93.98 40.64 180)
+      (effects (font (size 1.27 1.27)) (justify left))
+    )
+    (pin "3V_REG" output (at 118.11 40.64 0)
+      (effects (font (size 1.27 1.27)) (justify right))
+    )
+    (instances
+      (project "gkos_pebble"
+        (path "/ab6fff6e-44fa-4992-ab9d-8d9a7df4367d" (page "2"))
+      )
+    )
+  )
+  (sheet (at 190.5 129.54) (size 21.59 20.32) (fields_autoplaced)
+    (stroke (width 0.1524) (type solid))
+    (fill (color 255 255 194 1.0000))
+    (property "Sheetname" "lcd" (at 190.5 128.8284 0)
+      (effects (font (size 1.27 1.27)) (justify left bottom))
+    )
+    (property "Sheetfile" "lcd.kicad_sch" (at 190.5 150.4446 0)
+      (effects (font (size 1.27 1.27)) (justify left top))
+    )
+    (instances
+      (project "gkos_pebble"
+        (path "/ab6fff6e-44fa-4992-ab9d-8d9a7df4367d" (page "6"))
+      )
+    )
+  )
+  (sheet (at 147.32 50.8) (size 29.21 20.32) (fields_autoplaced)
+    (stroke (width 0.1524) (type solid))
+    (fill (color 255 255 194 1.0000))
+    (property "Sheetname" "ble" (at 147.32 50.0884 0)
+      (effects (font (size 1.27 1.27)) (justify left bottom))
+    )
+    (property "Sheetfile" "ble.kicad_sch" (at 147.32 71.7046 0)
+      (effects (font (size 1.27 1.27)) (justify left top))
+    )
+    (instances
+      (project "gkos_pebble"
+        (path "/ab6fff6e-44fa-4992-ab9d-8d9a7df4367d" (page "4"))
+      )
+    )
+  )
   (sheet_instances

Commit message: big commit with power and inputs
Other:
- sheet inputs ports: added EXT_~{RST}, KEY_A, KEY_B, KEY_C, KEY_D, KEY_E, KEY_F, MOUSE_1A, MOUSE_1B, MOUSE_2A, MOUSE_2B, MOUSE_3A, MOUSE_3B, TP_RDY, TP_SCL, TP_SDA, TP_~{RST}; removed none
- sheet power ports: added VUSB; removed USB_VBUS
Changed lines of the file:
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@@
     (comment 1 "main sheet")
   )
-  (text_box "- BLE module\n- RP2040 MCU\n- USB-C connection + TVS\n- keyboard switches\n- mouse buttons\n- touchpad\n- memory LCD"
-    (at 24.13 153.67 0) (size 50.8 25.4)
+  (wire (pts (xy 123.19 40.64) (xy 123.19 36.83))
+    (stroke (width 0) (type default))
+  )
+  (wire (pts (xy 118.11 40.64) (xy 123.19 40.64))
+    (stroke (width 0) (type default))
+  )
+  (text_box "- BLE module\n- RP2040 MCU\n- USB-C connection + TVS\n- memory LCD"
+    (at 24.13 153.67 0) (size 50.8 15.24)
     (stroke (width 0) (type default) (color 132 0 0 1))
     (fill (type color) (color 255 255 194 1))
@@
   (text "integration todo" (at 24.13 152.4 0)
     (effects (font (size 3 3) (thickness 0.6) bold italic (color 132 0 0 1)) (justify left bottom))
+  )
+  (symbol (lib_id "power:+3V0") (at 123.19 36.83 0) (unit 1)
+    (in_bom yes) (on_board yes) (dnp no)
+    (property "Reference" "#PWR02" (at 123.19 40.64 0)
+      (effects (font (size 1.27 1.27)) hide)
+    )
+    (property "Value" "+3V0" (at 123.19 33.02 0)
+      (effects (font (size 1.27 1.27)))
+    )
+    (property "Footprint" "" (at 123.19 36.83 0)
+      (effects (font (size 1.27 1.27)) hide)
+    )
+    (property "Datasheet" "" (at 123.19 36.83 0)
+      (effects (font (size 1.27 1.27)) hide)
+    )
+    (pin "1")
+    (instances
+      (project "gkos_pebble"
+        (path "/ab6fff6e-44fa-4992-ab9d-8d9a7df4367d"
+          (reference "#PWR02") (unit 1)
+        )
+      )
+    )
   )
   (sheet (at 127 114.3) (size 27.94 20.32) (fields_autoplaced)
@@
     )
   )
-  (sheet (at 92.71 72.39) (size 27.94 20.32) (fields_autoplaced)
+  (sheet (at 57.15 74.93) (size 15.24 53.34) (fields_autoplaced)
     (stroke (width 0.1524) (type solid))
     (fill (color 255 255 194 1.0000))
-    (property "Sheetname" "inputs" (at 92.71 71.6784 0)
+    (property "Sheetname" "inputs" (at 57.15 74.2184 0)
       (effects (font (size 1.27 1.27)) (justify left bottom))
     )
-    (property "Sheetfile" "inputs.kicad_sch" (at 92.71 93.2946 0)
-      (effects (font (size 1.27 1.27)) (justify left top))
+    (property "Sheetfile" "inputs.kicad_sch" (at 57.15 128.8546 0)
+      (effects (font (size 1.27 1.27)) (justify left top) hide)
+    )
+    (pin "KEY_D" output (at 72.39 85.09 0)
+      (effects (font (size 1.27 1.27)) (justify right))
+    )
+    (pin "KEY_C" output (at 72.39 82.55 0)
+      (effects (font (size 1.27 1.27)) (justify right))
+    )
+    (pin "KEY_E" output (at 72.39 87.63 0)
+      (effects (font (size 1.27 1.27)) (justify right))
+    )
+    (pin "KEY_F" output (at 72.39 90.17 0)
+      (effects (font (size 1.27 1.27)) (justify right))
+    )
+    (pin "KEY_B" output (at 72.39 80.01 0)
+      (effects (font (size 1.27 1.27)) (justify right))
+    )
+    (pin "KEY_A" output (at 72.39 77.47 0)
+      (effects (font (size 1.27 1.27)) (justify right))
+    )
+    (pin "MOUSE_3B" output (at 72.39 107.95 0)
+      (effects (font (size 1.27 1.27)) (justify right))
+    )
+    (pin "MOUSE_3A" output (at 72.39 105.41 0)
+      (effects (font (size 1.27 1.27)) (justify right))
+    )
+    (pin "MOUSE_2B" output (at 72.39 102.87 0)
+      (effects (font (size 1.27 1.27)) (justify right))
+    )
+    (pin "MOUSE_2A" output (at 72.39 100.33 0)
+      (effects (font (size 1.27 1.27)) (justify right))
+    )
+    (pin "EXT_~{RST}" output (at 72.39 125.73 0)
+      (effects (font (size 1.27 1.27)) (justify right))
+    )
+    (pin "TP_~{RST}" input (at 72.39 120.65 0)
+      (effects (font (size 1.27 1.27)) (justify right))
+    )
+    (pin "TP_SDA" bidirectional (at 72.39 115.57 0)
+      (effects (font (size 1.27 1.27)) (justify right))
+    )
+    (pin "TP_SCL" input (at 72.39 113.03 0)
+      (effects (font (size 1.27 1.27)) (justify right))
+    )
+    (pin "TP_RDY" output (at 72.39 118.11 0)
+      (effects (font (size 1.27 1.27)) (justify right))
+    )
+    (pin "MOUSE_1B" output (at 72.39 97.79 0)
+      (effects (font (size 1.27 1.27)) (justify right))
+    )
+    (pin "MOUSE_1A" output (at 72.39 95.25 0)
+      (effects (font (size 1.27 1.27)) (justify right))
     )
     (instances
@@
     )
   )
-  (sheet (at 93.98 38.1) (size 24.13 5.08) (fields_autoplaced)
+  (sheet (at 99.06 38.1) (size 19.05 5.08) (fields_autoplaced)
     (stroke (width 0.1524) (type solid))
     (fill (color 255 255 194 1.0000))
-    (property "Sheetname" "power" (at 93.98 37.3884 0)
+    (property "Sheetname" "power" (at 99.06 37.3884 0)
       (effects (font (size 1.27 1.27)) (justify left bottom))
     )
-    (property "Sheetfile" "power.kicad_sch" (at 93.98 43.7646 0)
-      (effects (font (size 1.27 1.27)) (justify left top))
-    )
-    (pin "USB_VBUS" input (at 93.98 40.64 180)
-      (effects (font (size 1.27 1.27)) (justify left))
+    (property "Sheetfile" "power.kicad_sch" (at 99.06 43.7646 0)
+      (effects (font (size 1.27 1.27)) (justify left top) hide)
     )
     (pin "3V_REG" output (at 118.11 40.64 0)
       (effects (font (size 1.27 1.27)) (justify right))
     )
+    (pin "VUSB" input (at 99.06 40.64 180)
+      (effects (font (size 1.27 1.27)) (justify left))
+    )
     (instances

Commit message: schema functionally done
Parts:
- added J4: 10129383-906002BLF, Connector_PinHeader_2.54mm:PinHeader_2x03_P2.54mm_Vertical_SMD, symbol Connector_Generic:Conn_02x03_Odd_Even
Connections:
- new net SWCLK_A: J4.2 (Pin_2)
- new net SWCLK_B: J4.6 (Pin_6)
- new net SWCLK_IN: J4.4 (Pin_4)
- new net SWD_A: J4.1 (Pin_1)
- new net SWD_B: J4.5 (Pin_5)
- new net SWD_IN: J4.3 (Pin_3)
Other:
- added sheet connectors (connectors.kicad_sch)
- sheet ble ports: added BLE_RESET, BLE_SCL, BLE_SDA, SWCLK, SWD; removed none
- sheet inputs ports: added MENU, ~{EXT_RST}, ~{USB_BOOT}; removed EXT_~{RST}
- sheet lcd ports: added LCD_COMIN, LCD_SCLK, LCD_SCS, LCD_SI; removed none
- sheet mcu ports: added KEY_A, KEY_B, KEY_C, KEY_D, KEY_E, KEY_F, LCD_COMIN, LCD_SCLK, LCD_SCS, LCD_SI, MENU, MOUSE_1A, MOUSE_1B, MOUSE_2A, MOUSE_2B, MOUSE_3A, MOUSE_3B, SCL, SDA, SWCLK, SWD, TP_RDY, USB_D+, USB_D-, ~{RST}, ~{USB_BOOT}; removed none
- sheet power ports: added 3V0_REG, 3V3_REG; removed 3V_REG
- note added: "I^{2}C"
- note added: "SPI"
- note added: "SWD"
- note added: "SWD target selection"
- note added: "USB 2.0"
- note removed: "integration todo"

Commit message: reannotation
Parts:
- renumbered J4 to J1
Changed lines of the file:
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@@
   (symbol (lib_id "Connector_Generic:Conn_02x03_Odd_Even") (at 194.31 143.51 0) (unit 1)
     (in_bom yes) (on_board yes) (dnp no)
-    (property "Reference" "J4" (at 195.58 138.43 0)
+    (property "Reference" "J1" (at 195.58 138.43 0)
       (effects (font (size 1.27 1.27)))
     )
@@
       (project "gkos_pebble"
         (path "/ab6fff6e-44fa-4992-ab9d-8d9a7df4367d"
-          (reference "J4") (unit 1)
+          (reference "J1") (unit 1)
         )
       )
@@
   (symbol (lib_id "power:+3V0") (at 158.75 58.42 0) (unit 1)
     (in_bom yes) (on_board yes) (dnp no)
-    (property "Reference" "#PWR010" (at 158.75 62.23 0)
+    (property "Reference" "#PWR02" (at 158.75 62.23 0)
       (effects (font (size 1.27 1.27)) hide)
     )
@@
       (project "gkos_pebble"
         (path "/ab6fff6e-44fa-4992-ab9d-8d9a7df4367d"
-          (reference "#PWR010") (unit 1)
+          (reference "#PWR02") (unit 1)
         )
       )
@@
   (symbol (lib_id "power:+3V3") (at 151.13 58.42 0) (unit 1)
     (in_bom yes) (on_board yes) (dnp no)
-    (property "Reference" "#PWR02" (at 151.13 62.23 0)
+    (property "Reference" "#PWR01" (at 151.13 62.23 0)
       (effects (font (size 1.27 1.27)) hide)
     )
@@
       (project "gkos_pebble"
         (path "/ab6fff6e-44fa-4992-ab9d-8d9a7df4367d"
-          (reference "#PWR02") (unit 1)
+          (reference "#PWR01") (unit 1)
         )
       )

Commit message: schematic cleanup
Other:
- moved on the sheet: J1
Changed lines of the file:
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@@
   (title_block
     (title "gkos pebble")
-    (date "2024-03-23")
+    (date "2024-03-25")
     (rev "1")
     (company "minteyay")
@@
     (stroke (width 0) (type default))
   )
-  (wire (pts (xy 177.8 143.51) (xy 189.23 143.51))
+  (wire (pts (xy 179.07 140.97) (xy 190.5 140.97))
     (stroke (width 0) (type default))
   )
@@
     (stroke (width 0) (type default))
   )
-  (wire (pts (xy 201.93 143.51) (xy 213.36 143.51))
+  (wire (pts (xy 203.2 140.97) (xy 214.63 140.97))
     (stroke (width 0) (type default))
   )
@@
     (stroke (width 0) (type default))
   )
-  (wire (pts (xy 201.93 140.97) (xy 213.36 140.97))
+  (wire (pts (xy 203.2 138.43) (xy 214.63 138.43))
     (stroke (width 0) (type default))
   )
@@
     (stroke (width 0) (type default))
   )
-  (wire (pts (xy 177.8 146.05) (xy 189.23 146.05))
+  (wire (pts (xy 179.07 143.51) (xy 190.5 143.51))
     (stroke (width 0) (type default))
   )
@@
     (stroke (width 0) (type default))
   )
-  (wire (pts (xy 177.8 140.97) (xy 189.23 140.97))
-    (stroke (width 0) (type default))
-  )
-  (wire (pts (xy 201.93 146.05) (xy 213.36 146.05))
+  (wire (pts (xy 179.07 138.43) (xy 190.5 138.43))
+    (stroke (width 0) (type default))
+  )
+  (wire (pts (xy 203.2 143.51) (xy 214.63 143.51))
     (stroke (width 0) (type default))
   )
@@
   )
   (text_box ""
-    (at 175.26 135.89 0) (size 40.64 15.24)
+    (at 175.26 130.81 0) (size 43.18 20.32)
     (stroke (width 0) (type dash) (color 132 0 0 1))
     (fill (type none))
     (effects (font (size 1.27 1.27)) (justify left top))
   )
-  (text "SWD" (at 177.8 91.44 0)
+  (text "SWD" (at 178.435 91.44 0)
     (effects (font (size 1.8 1.8) (thickness 0.4) bold italic (color 204 102 0 1)) (justify left bottom))
   )
@@
     (effects (font (size 1.8 1.8) (thickness 0.4) bold italic (color 204 102 0 1)) (justify left bottom))
   )
-  (text "SPI" (at 151.13 104.14 0)
-    (effects (font (size 1.8 1.8) (thickness 0.4) bold italic (color 204 102 0 1)) (justify left bottom))
-  )
-  (text "USB 2.0" (at 119.38 77.47 0)
-    (effects (font (size 1.8 1.8) (thickness 0.4) bold italic (color 204 102 0 1)) (justify left bottom))
-  )
-  (text "SWD target selection" (at 175.26 134.62 0)
+  (text "SPI" (at 153.035 104.775 0)
+    (effects (font (size 1.8 1.8) (thickness 0.4) bold italic (color 204 102 0 1)) (justify left bottom))
+  )
+  (text "USB 2.0" (at 119.38 76.835 0)
+    (effects (font (size 1.8 1.8) (thickness 0.4) bold italic (color 204 102 0 1)) (justify left bottom))
+  )
+  (text "SWD target selection" (at 175.26 129.54 0)
     (effects (font (size 2 2) (thickness 0.4) bold italic (color 132 0 0 1)) (justify left bottom))
   )
@@
     (effects (font (size 1.8 1.8) (thickness 0.4) bold italic (color 204 102 0 1)) (justify left bottom))
   )
-  (text "I^{2}C" (at 179.07 71.12 0)
+  (text "I^{2}C" (at 179.705 71.12 0)
     (effects (font (size 1.8 1.8) (thickness 0.36) bold italic (color 204 102 0 1)) (justify left bottom))
   )
-  (text "SWD" (at 151.13 91.44 0)
-    (effects (font (size 1.8 1.8) (thickness 0.4) bold italic (color 204 102 0 1)) (justify left bottom))
-  )
-  (text "I^{2}C" (at 151.13 134.62 0)
+  (text "SWD" (at 152.4 91.44 0)
+    (effects (font (size 1.8 1.8) (thickness 0.4) bold italic (color 204 102 0 1)) (justify left bottom))
+  )
+  (text "I^{2}C" (at 151.765 135.255 0)
     (effects (font (size 1.8 1.8) (thickness 0.4) bold italic (color 204 102 0 1)) (justify left bottom))
   )
@@
     (effects (font (size 1.27 1.27)) (justify right bottom))
   )
-  (label "SWCLK_A" (at 213.36 140.97 180) (fields_autoplaced)
+  (label "SWCLK_A" (at 214.63 138.43 180) (fields_autoplaced)
     (effects (font (size 1.27 1.27)) (justify right bottom))
   )
@@
     (effects (font (size 1.27 1.27)) (justify right bottom))
   )
-  (label "SWD_IN" (at 177.8 143.51 0) (fields_autoplaced)
-    (effects (font (size 1.27 1.27)) (justify left bottom))
-  )
-  (label "SWD_A" (at 177.8 140.97 0) (fields_autoplaced)
+  (label "SWD_IN" (at 179.07 140.97 0) (fields_autoplaced)
+    (effects (font (size 1.27 1.27)) (justify left bottom))
+  )
+  (label "SWD_A" (at 179.07 138.43 0) (fields_autoplaced)
     (effects (font (size 1.27 1.27)) (justify left bottom))
   )
@@
     (effects (font (size 1.27 1.27)) (justify right bottom))
   )
-  (label "SWD_B" (at 177.8 146.05 0) (fields_autoplaced)
-    (effects (font (size 1.27 1.27)) (justify left bottom))
-  )
-  (label "SWCLK_IN" (at 213.36 143.51 180) (fields_autoplaced)
-    (effects (font (size 1.27 1.27)) (justify right bottom))
-  )
-  (label "SWCLK_B" (at 213.36 146.05 180) (fields_autoplaced)
-    (effects (font (size 1.27 1.27)) (justify right bottom))
-  )
-  (symbol (lib_id "Connector_Generic:Conn_02x03_Odd_Even") (at 194.31 143.51 0) (unit 1)
+  (label "SWD_B" (at 179.07 143.51 0) (fields_autoplaced)
+    (effects (font (size 1.27 1.27)) (justify left bottom))
+  )
+  (label "SWCLK_IN" (at 214.63 140.97 180) (fields_autoplaced)
+    (effects (font (size 1.27 1.27)) (justify right bottom))
+  )
+  (label "SWCLK_B" (at 214.63 143.51 180) (fields_autoplaced)
+    (effects (font (size 1.27 1.27)) (justify right bottom))
+  )
+  (symbol (lib_id "Connector_Generic:Conn_02x03_Odd_Even") (at 195.58 140.97 0) (unit 1)
     (in_bom yes) (on_board yes) (dnp no)
-    (property "Reference" "J1" (at 195.58 138.43 0)
+    (property "Reference" "J1" (at 196.85 135.255 0)
       (effects (font (size 1.27 1.27)))
     )
-    (property "Value" "10129383-906002BLF" (at 195.58 148.59 0)
+    (property "Value" "10129383-906002BLF" (at 197.485 146.685 0)
       (effects (font (size 1.27 1.27)))
     )
-    (property "Footprint" "Connector_PinHeader_2.54mm:PinHeader_2x03_P2.54mm_Vertical_SMD" (at 194.31 143.51 0)
-      (effects (font (size 1.27 1.27)) hide)
-    )
-    (property "Datasheet" "~" (at 194.31 143.51 0)
+    (property "Footprint" "Connector_PinHeader_2.54mm:PinHeader_2x03_P2.54mm_Vertical_SMD" (at 195.58 140.97 0)
+      (effects (font (size 1.27 1.27)) hide)
+    )
+    (property "Datasheet" "~" (at 195.58 140.97 0)
       (effects (font (size 1.27 1.27)) hide)
     )
@@
     )
   )
-  (sheet (at 83.82 59.69) (size 15.24 20.32) (fields_autoplaced)
+  (sheet (at 83.82 59.69) (size 15.24 20.32)
     (stroke (width 0.1524) (type solid) (color 132 0 0 1))
     (fill (color 255 255 194 1.0000))
-    (property "Sheetname" "connectors" (at 83.82 58.9784 0)
+    (property "Sheetname" "connectors" (at 83.82 59.055 0)
       (effects (font (size 1.27 1.27)) (justify left bottom))
     )
@@
     )
   )
-  (sheet (at 121.92 82.55) (size 27.94 58.42) (fields_autoplaced)
+  (sheet (at 121.92 82.55) (size 27.94 58.42)
     (stroke (width 0.1524) (type solid))
     (fill (color 255 255 194 1.0000))
-    (property "Sheetname" "mcu" (at 121.92 81.8384 0)
+    (property "Sheetname" "mcu" (at 121.92 81.915 0)
       (effects (font (size 1.27 1.27)) (justify left bottom))
     )
@@
     )
   )
-  (sheet (at 83.82 90.17) (size 15.24 60.96) (fields_autoplaced)
+  (sheet (at 83.82 90.17) (size 15.24 60.96)
     (stroke (width 0.1524) (type solid))
     (fill (color 255 255 194 1.0000))
-    (property "Sheetname" "inputs" (at 83.82 89.4584 0)
+    (property "Sheetname" "inputs" (at 83.82 89.535 0)
       (effects (font (size 1.27 1.27)) (justify left bottom))
     )
@@
     )
   )
-  (sheet (at 127 59.69) (size 19.05 7.62) (fields_autoplaced)
+  (sheet (at 127 59.69) (size 19.05 7.62)
     (stroke (width 0.1524) (type solid))
     (fill (color 255 255 194 1.0000))
-    (property "Sheetname" "power" (at 127 58.9784 0)
+    (property "Sheetname" "power" (at 127 59.055 0)
       (effects (font (size 1.27 1.27)) (justify left bottom))
     )
